File: hardware/Ankle_Sensor_V1.kicad_pcb (KiCad board)
At the start: 4 copper layers, 30 x 51.6 mm, 69 parts, among them J1 TYPE-C-31-M-12, J2 JST_SH_3P_PACK_NTC, J3 SWD_POGO_6, Q1 AO3400A, Q2 AO3400A, SW1 SKQGABE010, U1 BQ25185DLHR, U2 TPS7A2030PDBVR, U3 MDBT50Q-P1MV2, U4 LSM6DSV32XTR, U5 W25Q01JVZEIQ_128MiB, U6 USBLC6-2SC6, U7 TLV7042DGKR, U8 TLV803EA26DBZR, Y1 32.768kHz CL7pF

Commit message: update
Parts:
- moved U6 4.30 mm to (71.6, 93.3)
- moved R25 3.60 mm to (74.8, 92.2)
Connections:
- R24 pad 2: GND -> +3V0
Routing:
- net USB_DP_CONN: track 18.7 -> 13.0 mm, vias 0 -> 2
- net USB_DN_CONN: track 20.6 -> 15.6 mm
- net USB_DP: track 35.7 -> 31.2 mm
- net VBUS: track 59.3 -> 54.9 mm
- net USB_DN: track 36.1 -> 33.0 mm
- net GND: track 42.1 -> 41.4 mm, vias 53 -> 52
- net +3V0: track 24.9 -> 25.5 mm, vias 32 -> 33
- net SW_RETURN: track 8.03 -> 8.46 mm, vias 0 -> 2
