File: hardware/Ankle_Sensor_V1.kicad_pcb (KiCad board)
At the start: 4 copper layers, 30 x 51.6 mm, 69 parts, among them J1 TYPE-C-31-M-12, J2 JST_SH_3P_PACK_NTC, J3 SWD_POGO_6, Q1 AO3400A, Q2 AO3400A, SW1 SKQGABE010, U1 BQ25185DLHR, U2 TPS7A2030PDBVR, U3 MDBT50Q-P1MV2, U4 LSM6DSV32XTR, U5 W25Q01JVZEIQ_128MiB, U6 USBLC6-2SC6, U7 TLV7042DGKR, U8 TLV803EA26DBZR, Y1 32.768kHz CL7pF

Commit message: update
Parts:
- C9: value 4.7u 10V X5R -> 10u 10V X5R
Changed lines of the file:
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@@
 			)
 		)
-		(property "Value" "4.7u 10V X5R"
+		(property "Value" "10u 10V X5R"
 			(at 0 1.43 0)
 			(layer "F.Fab")
@@
 			)
 		)
-		(property "MPN" "CL10A475KP8NNNC"
+		(property "MPN" "CL10A106KP8NNNC"
 			(at 0 0 0)
 			(layer "F.SilkS")
@@
 			)
 		)
-		(property "JLCPCB" "C1705"
+		(property "JLCPCB" "C19702"
 			(at 0 0 0)
 			(layer "F.SilkS")
@@
 			)
 		)
-		(property "Note" ""
+		(property "Note" "10uF nominal aligns supply reference; Ceff is not10uF guaranteed; see docs/production_caps_A1.md"
 			(at 0 0 0)
 			(layer "F.SilkS")
