File: hardware/temperature.kicad_sch (KiCad schematic)
At the start: 13 parts, among them Q1 AO3400A, Q2 AO3400A, U7 TLV7042DGKR, U8 TLV803EA26DBZR

Commit message: update
Parts:
- R24: Note Q2 defaultsOFF with GPIOHiZ -> 100k pull-up: Q2 inhibits charging during MCU reset/HiZ; LO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
Connections:
- net +3V0: now also R24.2
- net GND: no longer R24.2
Other:
- note added: "P1.14 HIGH/HiZ/reset=inhibit via Q2; LOW releases to hardware window."
- note removed: "Firmware P1.14 HIGH=inhibit viaQ2; LOW/HiZ permits hardware control."
Changed lines of the file:
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@@
 (kicad_sch (version 20231120) (generator "ankle_sensor_review_generator") (paper "A3")
-(title_block (title "Ankle Sensor V1 / temperature") (date "2026-10-28") (rev "A1-WIP") (comment 1 "WORK IN PROGRESS - SEE CURRENT ERC/DRC REPORTS"))
+(title_block (title "Ankle Sensor V1 / temperature") (date "2026-10-29") (rev "A1-AUDIT") (comment 1 "AUDIT REVIEW - SEE CURRENT ERC/DRC REPORTS"))
 (text "INDEPENDENT BATTERY NTC WINDOW - REVIEW DRAFT" (at 25 17 0) (effects (font (size 1.05 1.05)) (justify left)))
 (text "NTC103AT-2 /10k B3435 must be on CELL. No10k bypass resistor is permitted." (at 25 25 0) (effects (font (size 1.05 1.05)) (justify left)))
-(text "Firmware P1.14 HIGH=inhibit viaQ2; LOW/HiZ permits hardware control." (at 25 33 0) (effects (font (size 1.05 1.05)) (justify left)))
+(text "P1.14 HIGH/HiZ/reset=inhibit via Q2; LOW releases to hardware window." (at 25 33 0) (effects (font (size 1.05 1.05)) (justify left)))
 (text "U8 holdsALLOWlow during reference startup. See tolerance calculation and tests." (at 25 281 0) (effects (font (size 1.05 1.05)) (justify left)))
 (text "Pack acceptance: R0C>=24k, R45C<=5.20k, monotonic. Physical qualification required." (at 25 289 0) (effects (font (size 1.05 1.05)) (justify left)))
@@
 (property "JLCPCB" "C25741" (at 165.1 250.19 0) (effects (font (size 1 1)) hide))
 (property "ReviewStatus" "REVIEW" (at 165.1 250.19 0) (effects (font (size 1 1)) hide))
-(property "Note" "Q2 defaultsOFF with GPIOHiZ" (at 165.1 250.19 0) (effects (font (size 1 1)) hide))
+(property "Note" "100k pull-up: Q2 inhibits charging during MCU reset/HiZ; LOW releases hardware window" (at 165.1 250.19 0) (effects (font (size 1 1)) hide))
 (pin "1")
 (pin "2")
@@
 (global_label "CHG_INHIBIT" (shape passive) (at 152.4 250.19 0) (effects (font (size 0.9 0.9)) (justify left)) (property "Intersheetrefs" "${INTERSHEET_REFS}" (at 152.4 250.19 0) (effects (font (size 1 1)) hide)))
 (wire (pts (xy 170.18 250.19) (xy 177.8 250.19)) (stroke (width 0) (type default)))
-(global_label "GND" (shape passive) (at 177.8 250.19 180) (effects (font (size 0.9 0.9)) (justify left)) (property "Intersheetrefs" "${INTERSHEET_REFS}" (at 177.8 250.19 0) (effects (font (size 1 1)) hide)))
+(global_label "+3V0" (shape passive) (at 177.8 250.19 180) (effects (font (size 0.9 0.9)) (justify left)) (property "Intersheetrefs" "${INTERSHEET_REFS}" (at 177.8 250.19 0) (effects (font (size 1 1)) hide)))
 (symbol (lib_id "AnkleSensor:C") (at 165.1 209.55 0) (unit 1) (in_bom yes) (on_board yes) (dnp no)
 (property "Reference" "C19" (at 165.1 203.44500000000002 0) (effects (font (size 1 1))))
