File: hardware/mcu.kicad_sch (KiCad schematic)
At the start: 9 parts, among them U3 MDBT50Q-P1MV2, Y1 32.768kHz CL7pF

Commit message: update
Parts:
- C9: value 4.7u 10V X5R -> 10u 10V X5R; JLCPCB C1705 -> C19702; MPN CL10A475KP8NNNC -> CL10A106KP8NNNC; Note (none) -> 10uF nominal aligns supply reference; Ceff is not10uF guara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
Changed lines of the file:
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@@
 (symbol (lib_id "AnkleSensor:C") (at 204.47 124.46 0) (unit 1) (in_bom yes) (on_board yes) (dnp no)
 (property "Reference" "C9" (at 204.47 118.35499999999999 0) (effects (font (size 1 1))))
-(property "Value" "4.7u 10V X5R" (at 204.47 120.755 0) (effects (font (size 0.9 0.9))))
+(property "Value" "10u 10V X5R" (at 204.47 120.755 0) (effects (font (size 0.9 0.9))))
 (property "Footprint" "AnkleSensor:C_0603_1608Metric" (at 204.47 124.46 0) (effects (font (size 1 1)) hide))
 (property "Datasheet" "" (at 204.47 124.46 0) (effects (font (size 1 1)) hide))
-(property "MPN" "CL10A475KP8NNNC" (at 204.47 124.46 0) (effects (font (size 1 1)) hide))
-(property "JLCPCB" "C1705" (at 204.47 124.46 0) (effects (font (size 1 1)) hide))
+(property "MPN" "CL10A106KP8NNNC" (at 204.47 124.46 0) (effects (font (size 1 1)) hide))
+(property "JLCPCB" "C19702" (at 204.47 124.46 0) (effects (font (size 1 1)) hide))
 (property "ReviewStatus" "REVIEW" (at 204.47 124.46 0) (effects (font (size 1 1)) hide))
-(property "Note" "" (at 204.47 124.46 0) (effects (font (size 1 1)) hide))
+(property "Note" "10uF nominal aligns supply reference; Ceff is not10uF guaranteed; see docs/production_caps_A1.md" (at 204.47 124.46 0) (effects (font (size 1 1)) hide))
 (pin "1")
 (pin "2")
